File: _autosave-figleaf.kicad_pcb (KiCad board)
At the start: 2 copper layers, 110.8 x 98.5 mm, 5 parts, among them U1 Nice_Nano_V2

Commit message: progress pcb
Routing:
- net col_1: track 49.4 -> 57.1 mm, vias 0 -> 1
- net col_0: track 73.9 -> 80.4 mm, vias 0 -> 1
- added copper zone on F.Cu, net GND_L
