File: _autosave-figleaf-integrated.kicad_pcb (KiCad board)
At the start: 2 copper layers, 145 x 105 mm, 61 parts, among them J2 HRO_TYPE-C-31-M-14, J3 Battery, J9 TC2030_SWD, Q2 2N7002, SW1 PWR, SW2 RST, U1 SRV05-4, U3 BQ24075, U8 nRF52840_moko_mk08

Commit message: prog
Parts:
- moved SW2 0.25 mm to (129.2, 14.0)
Routing:
- net Net-(J2-CC1): track 0.00 -> 7.58 mm, vias 0 -> 2
- net Net-(Q2-G): track 2.46 -> 7.98 mm, vias 0 -> 2
- net GND_L: vias 7 -> 8
