File: _autosave-figleaf-integrated.kicad_sch (KiCad schematic)
At the start: 71 parts, among them J1 Conn_01x02_Pin, J2 HRO_TYPE-C-31-M-14, J3 Battery, J9 TC2030_SWD, Q2 2N7002, SW1 PWR, SW2 RST, U1 SRV05-4, U10 MAX17048, U3 BQ24075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

Commit message: move jst + add optional battery pad
Parts:
- J1: footprint Connector_PinHeader_1.27mm:PinHeader_1x02_P1.27mm_Vertical -> (none)
Changed lines of the file:
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@@
 			)
 		)
-		(property "Footprint" "Connector_PinHeader_1.27mm:PinHeader_1x02_P1.27mm_Vertical"
+		(property "Footprint" ""
 			(at 222.25 57.15 0)
 			(effects
