File: _autosave-figleaf-integrated.kicad_sch (KiCad schematic)
At the start: 70 parts, among them J1 Conn_01x02_Pin, J2 HRO_TYPE-C-31-M-14, J3 Battery, J9 TC2030_SWD, Q2 2N7002, SW1 PWR, SW2 RST, U1 SRV05-4, U10 MAX17048, U3 BQ24075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

Commit message: all routed
Changed lines of the file:
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@@
+	)
+	(junction
+		(at 231.14 39.37)
+		(diameter 0)
+		(color 0 0 0 0)
 	)
 	(junction
@@
 	)
 	(junction
-		(at 231.14 39.37)
-		(diameter 0)
-		(color 0 0 0 0)
-	)
-	(junction
 		(at 26.67 68.58)
 		(diameter 0)
@@
 	(wire
 		(pts
+			(xy 231.14 39.37) (xy 236.22 39.37)
+		)
+		(stroke
+			(width 0)
+			(type default)
+		)
+	)
+	(wire
+		(pts
 			(xy 349.25 167.64) (xy 354.33 167.64)
 		)
@@
 	(wire
 		(pts
+			(xy 243.84 44.45) (xy 261.62 44.45)
+		)
+		(stroke
+			(width 0)
+			(type default)
+		)
+	)
+	(wire
+		(pts
 			(xy 293.37 152.4) (xy 293.37 157.48)
 		)
@@
 	(wire
 		(pts
-			(xy 261.62 44.45) (xy 243.84 44.45)
-		)
-		(stroke
-			(width 0)
-			(type default)
-		)
-	)
-	(wire
-		(pts
 			(xy 369.57 127) (xy 369.57 132.08)
 		)
@@
 		)
 	)
-	(wire
-		(pts
-			(xy 231.14 39.37) (xy 236.22 39.37)
-		)
-		(stroke
-			(width 0)
-			(type default)
-		)
-	)
