File: side.kicad_sch (KiCad schematic)
At the start: 76 parts, among them J1 Conn_01x02_Pin, J2 HRO_TYPE-C-31-M-14, J3 Battery, J9 TC2030_SWD, Q2 2N7002, SW1 PWR, SW2 RST, U1 SRV05-4, U10 MAX17048, U3 BQ24075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

Commit message: Update pwr switch symbol
Parts:
- SW1: symbol kigraz:SW_Push_SPDT -> kigraz:SW_SPDT_MP
Changed lines of the file:
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@@
 	)
 	(symbol
-		(lib_id "kigraz:SW_Push_SPDT")
+		(lib_id "kigraz:SW_SPDT_MP")
 		(at 256.54 33.02 0)
 		(unit 1)
@@
 			)
 		)
-		(property "Datasheet" ""
-			(at 256.54 33.02 0)
+		(property "Datasheet" "https://tech.alpsalpine.com/e/products/detail/SSSS811101/"
+			(at 257.048 41.656 0)
 			(hide yes)
 			(show_name no)
@@
 			)
 		)
-		(property "Description" "Momentary Switch, single pole double throw"
+		(property "Description" "Switch, single pole double throw"
 			(at 257.556 26.924 0)
 			(hide yes)
